File: LoraGateway.sch (EAGLE design)
At the start: 150 parts, among them IC1 TPS7A80, P1 LTST-C191KGKT, P2 LTST-C930KGKT, P3 LTST-C930KGKT, U1 SC283, U10 SE2435L, U2 SC560H, U4 STM32F401CDU6, U6 SX1257, U7 SX1257, X1 USB2-MICRO, X2 MCU Prog Header, X3 END4825A, X4 END4263A, X5 SMA-KE11

Commit message: old layout removed, Rpi-Zero Header added
Parts:
- removed C12, C13, C17, C18, C19, C20, C21: 100nF, rcl:C-EUC0402
- removed C14, C15: 4.7µF, rcl:C-EUC0603
- removed C16: 1µF, rcl:C-EUC0402
- removed C22: 56pF, rcl:C-EUC0402
- removed C75: 10nF, rcl:C-EUC0402
- removed D3, D4: RCLAMP0531T, LoRa Gateway:RCLAMP0531T
- removed FB5, FB6: (no value), LoRa Gateway:BLM15PG100SN1D0402
- removed IC1: TPS7A80, LoRa Gateway:TPS7A80
- removed JP1: SPI_Debug, pinhead:PINHD-1X6
- removed P1: LTST-C191KGKT, LoRa Gateway:LTST-C191KGKT
- removed R10: 10k, rcl:R-EU_R0402
- removed R11: 100, rcl:R-EU_R0402
- removed R3: 1k, rcl:R-EU_R0402
- removed R8, R9: 100k, rcl:R-EU_R0402
- removed S1, S2: KXT121LHS, LoRa Gateway:KXT121LHS
- removed U4: STM32F401CDU6, LoRa Gateway:STM32F401CDU6
- removed X2: MCU Prog Header, con-amp-micromatch:MICROMATCH-6
- added J1: RPI-ZERO-HEADER, LoRa Gateway:RPI-ZERO-HEADER
- added U3: (no value), LoRa Gateway:SC4212
- R1: value 0R -> 16k; OC_DIGIKEY 541-4062-1-ND -> 541-10KJCT-ND
- R2: value 0R -> 12k; OC_DIGIKEY 541-4062-1-ND -> 541-10KJCT-ND
Connections:
- removed net +3V3: C15.1, C16.1, C17.1, C18.1, C19.1, C20.1, C21.1, FB6.2, R9.2, S1.1, U4.VBAT, U4.VDD@1, U4.VDD@2, U4.VDD@3, U4.VDDA/VREF+
- removed net BOOT0: R8.2, S1.2, U4.BOOT0
- removed net D+: D4.1, R2.1, X1.D+
- removed net D-: D3.1, R1.1, X1.D-
- removed net I2C1_SCL: U4.PB7
- removed net I2C1_SDA: U4.PB6
- removed net N$10: P1.A, R3.1
- removed net N$33: R11.2, U4.PB0
- removed net N$5: C12.1, FB5.1, X2-5.S
- removed net NRST: C13.1, R9.1, S2.2, U4.NRST, X2-1.S
- removed net RADIO2_RST: U4.PA10
- removed net SPI2_MISO: U4.PB14
- removed net SPI2_MOSI: U4.PB15
- removed net SPI2_NSS: U4.PB12
- removed net SPI2_SCK: U4.PB13
- removed net SWCLK: U4.PA14, X2-4.S
- removed net SWDIO: U4.PA13, X2-6.S
- removed net TRACESWO: U4.PB3, X2-2.S
- removed net USB_DM: R1.2, U4.PA11
- removed net USB_DP: R2.2, U4.PA12
- removed net VCAP: C14.1, U4.VCAP1
- net +5V: no longer R3.2, U4.PA9
- net 133M_OUT_EN: no longer R10.2, U4.PB2
- net CLKO_B_32M: no longer U4.PH0-OSC_IN
- net FEM_EN: now also U3.EN; no longer C22.1, IC1.EN, R11.1
- net GND: now also R2.1, U3.GND; no longer C12.2, C13.2, C14.2, C15.2, C16.2, C17.2, C18.2, C19.2, C20.2, C21.2, C22.2, C75.2, D3.2, D4.2, IC1.GND, JP1.6, P1.C, R10.1, R8.1, S2.1, U4.VSS@1, U4.VSS@2, U4.VSS@3, U4.VSS@4, U4.VSSA/VREF-, X2-3.S
- net GPIO0: no longer U4.PB1
- net GPIO2: no longer U4.PA2
- net GPIO3: no longer U4.PA8
- net N$12: now also U3.VIN; no longer IC1.VIN
- net N$3: now also R1.1, R2.2, U3.FB; no longer C75.1, IC1.NR
- net PPS: no longer U4.PB10
- net RADIO_EN_A: no longer U4.PB8
- net RADIO_EN_B: no longer U4.PB9
- net RADIO_RST: no longer U4.PA0
- net RESET: no longer JP1.1, U4.PA3
- net RX_ON: no longer U4.PB5
- net SPI_MISO: no longer JP1.4, U4.PA6
- net SPI_MOSI: no longer JP1.5, U4.PA7
- net SPI_NSS: no longer JP1.2, U4.PA4
- net SPI_SCK: no longer JP1.3, U4.PA5
- net TX_ON: no longer U4.PB4
- net VCCDIG33: no longer FB5.2, FB6.1
- net VCCINT: now also R1.2, U3.VOUT; no longer IC1.SNS, IC1.VOUT
