File: layout/LoraGateway.sch (EAGLE design)
At the start: 124 parts, among them J1 RPI-ZERO-HEADER, P2 LTST-C930KGKT, P3 LTST-C930KGKT, U1 SC283, U10 SE2435L, U2 SC560H, U6 SX1257, U7 SX1257, X1 USB2-MICRO, X3 END4825A, X4 END4263A, X5 SMA-KE11

Commit message: Rpi-shield
Parts:
- removed P3: LTST-C930KGKT, LoRa Gateway:LTST-C930KGKT
- removed R19, R22: 100, rcl:R-EU_R0402
- added C12: 100nF, common:C-EU0402
- added C13: 56pF, rcl:C-EUC0402
- added P1, P5, P6, P7, P8: LTST-C930KGKT, LoRa Gateway:LTST-C930KGKT
- added R10, R11, R7, R8, R9: 470, rcl:R-EU_R0402
- added R3: EXB-N8V101JX, LoRa Gateway:EXB-N8V101JX
- added R6: 100, rcl:R-EU_R0402
- added U4: FGPMMOPA6H, LoRa Gateway:FGPMMOPA6H
- added X2: SMA-KE11, LoRa Gateway:SMA-KE11
- C1, C2, C3, C4: device rcl:C-EUC1206 -> common:C-EU1206
- C11, C23, C36, C5, C9: device rcl:C-EUC0805 -> common:C-EU0805
- C24, C26, C27, C28, C29, C30, C31, C32, C33, C35, C39, C40, C41, C42, C43, C44, C48, C49, C50, C51, C52, C55, C56, C59, C60, C61, C62, C63, C64, C65, C66, C67, C68, C69, C70, C71, C72, C73, C74: device rcl:C-EUC0402 -> common:C-EU0402
- C25, C34, C37, C38, C45, C46, C47, C53, C54, C58, C6: device rcl:C-EUC0603 -> common:C-EU0603
- J1: value RPI-ZERO-HEADER -> RPI-HEADER3B; device LoRa Gateway:RPI-ZERO-HEADER -> LoRa Gateway:RPI-HEADER3B
- R16, R17: value 470 -> 100; OC_DIGIKEY 311-470JRCT-ND -> 541-100ATCT-ND
- R18: value 100 -> 470; OC_DIGIKEY 541-100ATCT-ND -> 311-470JRCT-ND
Connections:
- removed net CLKO_B_32M: R22.2
- removed net GPIO0: U5.GPIO[0]
- removed net GPIO2: U5.GPIO[2]
- removed net GPIO3: U5.GPIO[3]
- removed net N$15 (its old number): P3.A, R17.2
- new net 3V3@1: J1.3V3@1
- new net N$10: R3.8, U5.HOST_SCK
- new net N$11: R3.7, U5.HOST_MISO
- new net N$33: R3.5, U5.HOST_CSN
- new net N$42: P1.A, R7.2
- new net N$5: R6.1, U5.SP_CLK_OUT
- new net N$51: U4.EX_ANT, X2.1
- new net N$66: P6.A, R9.2
- new net N$68: P7.A, R10.2
- new net N$69: P8.A, R11.2
- new net N$7: R11.1, U5.GPIO[0]
- new net N$71: R8.1, U5.GPIO[3]
- new net N$72: R18.2, U4.3DFIX
- new net N$73: U4.TX
- new net N$74: U4.RX
- new net N$75: C12.1, U4.!RESET, U4.VCC
- new net N$76: P2.A, R18.1
- new net N$8: R9.1, U5.GPIO[2]
- net +5V: now also J1.5V0@1, J1.5V0@2
- net CLKI: now also R6.2; no longer R18.2
- net CLKO_B: now also R17.2; no longer R19.2, R22.1
- net FEM_EN: now also R16.2; no longer U3.EN
- net GND: now also C12.2, C13.2, J1.GND@1, J1.GND@2, J1.GND@3, J1.GND@4, J1.GND@5, J1.GND@6, J1.GND@7, J1.GND@8, P1.C, P5.C, P6.C, P7.C, P8.C, U10.N/C@6, U4.GND@1, U4.GND@2, U4.GND@3, U4.GND@4, X2.GND; no longer P3.C
- net N$12: now also U3.EN
- net N$14: now also R3.6, U5.HOST_MOSI; no longer P2.A, R16.2
- net N$45: now also P5.A, R8.2; no longer R18.1, U5.SP_CLK_OUT
- net N$58: now also R17.1; no longer R19.1
- net PPS: now also J1.GEN5/GPIO24, U4.PPS
- net RADIO_RST: now also U5.RADIO_RST
- net RESET: now also J1.GEN/6GPIO25
- net RX_ON: now also R10.1; no longer R17.1
- net SPI_MISO: now also J1.GPIO9/MISO, R3.2; no longer U5.HOST_MISO
- net SPI_MOSI: now also J1.GPIO10/MOSI, R3.3; no longer U5.HOST_MOSI
- net SPI_NSS: now also J1.!CE0!/GPIO8, R3.4; no longer U5.HOST_CSN
- net SPI_SCK: now also J1.GPIO11/SCLK, R3.1; no longer U5.HOST_SCK
- net TX_ON: now also R7.1; no longer R16.1
- net VCCINT: now also C13.1, R16.1
Other:
- moved on the sheet: C10, C25, C26, C27, C30, C35, C36, C37, C5, C55, C59, C7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

Commit message: gps modul connected
Parts:
- removed C5: 1µF, common:C-EU0805
- removed D1, D2: RCLAMP0531T, LoRa Gateway:RCLAMP0531T
- removed FB1, FB2, FB3: (no value), LoRa Gateway:BLM15PG100SN1D0402
- removed X1: USB2-MICRO, LoRa Gateway:USB2-MICRO
- added R19: 0, rcl:R-EU_R0402
Connections:
- removed net N$6: D1.1, FB3.1, X1.GND
- removed net N$73: U4.TX
- removed net N$74: U4.RX
- removed net N$9: FB1.2, X1.SHIELD
- removed net VBUS: D2.1, FB2.1, X1.VCC
- new net 3V3@2: J1.3V3@2
- new net GPSRX: J1.TXD0/GPIO14, U4.RX
- new net GPSTX: J1.RXD0/GPIO15, U4.TX
- net +5V: no longer C5.2, FB2.2
- net GND: now also R19.1; no longer C5.1, D1.2, D2.2, FB1.1, FB3.2
- net N$75: now also R19.2
Other:
- moved on the sheet: C12, P2, R18
