File: layout/LoraGateway_pr.sch (EAGLE design)
At the start: 130 parts, among them J1 RPI-HEADER3B, U10 SE2435L, U2 FGPMMOPA6H, U4 SC283, U5 SC560H, U6 SX1257, U7 SX1257, X1 END4825A, X2 SMA-KE11, X3 END4263A, X4 SMA-KE11

Commit message: gateway routed
Parts:
- removed D8: BAT54XV2T1G, LoRa Gateway:BAT54XV2T1G
- removed D9: LXES15AAA1-153, LoRa Gateway:LXES15AAA1-153
- removed J1: RPI-HEADER3B, LoRa Gateway:RPI-HEADER3B
- removed R6: 100, common:R-EU0402
- removed R7: 470, common:R-EU0603
- removed U3: (no value), LoRa Gateway:SC4212
- added C65, C69: 3.3pF, rcl:C-EUC0402
- added C66: 33pF, rcl:C-EUC0402
- added C67: 7.5pF, rcl:C-EUC0402
- added C68: 1.5pF, rcl:C-EUC0402
- added C70, C72: 5.1pF, rcl:C-EUC0402
- added C71: 2.7pF, rcl:C-EUC0402
- added C73: 56pF, rcl:C-EUC0402
- added C74: 100nF, rcl:C-EUC0402
- added C75: 10nF, rcl:C-EUC0402
- added FB10: (no value), LoRa Gateway:BLM18PG121SH1D
- added FB6, FB7, FB8, FB9: (no value), LoRa Gateway:BLM15PG100SN1D0402
- added IC1: TPS7A80, LoRa Gateway:TPS7A80
- added JP1: SPI_Debug, pinhead:PINHD-1X6
- added P1: LTST-C191KGKT, LoRa Gateway:LTST-C191KGKT
- added P2, P3: LTST-C930KGKT, LoRa Gateway:LTST-C930KGKT
- added R26, R27: 49R9, rcl:R-EU_R0402
- added S1, S2: KXT121LHS, LoRa Gateway:KXT121LHS
- added X5: SMA-KE11, LoRa Gateway:SMA-KE11
- C1: value 10µF -> 22uF; device common:C-EU0805 -> rcl:C-EUC1206; OC_DIGIKEY 1276-2399-1-ND -> 445-6001-1-ND
- C10, C7: value 100nF -> 10uF; device common:C-EU0402 -> rcl:C-EUC0805; OC_DIGIKEY 478-7888-1-ND -> 1276-2399-1-ND
- C11, C9: value 100nF -> 1uF; device common:C-EU0402 -> rcl:C-EUC0805; OC_DIGIKEY 478-7888-1-ND -> 490-1691-1-ND
- C12, C30, C41, C42: value 1µF -> 100nF; device common:C-EU0402 -> rcl:C-EUC0402; OC_DIGIKEY 1276-1076-1-ND -> 478-7888-1-ND
- C13, C22, C33, C35, C39, C8: device common:C-EU0402 -> rcl:C-EUC0402
- C14: value 10µF -> 4.7µF; device common:C-EU0805 -> rcl:C-EUC0603; OC_DIGIKEY 1276-2399-1-ND -> 1276-1905-1-ND
- C15: value 100nF -> 4.7µF; device common:C-EU0402 -> rcl:C-EUC0603; OC_DIGIKEY 478-7888-1-ND -> 1276-1905-1-ND
- C16: device common:C-EU0603 -> rcl:C-EUC0402; OC_DIGIKEY 490-1543-1-ND -> 478-4596-1-ND
- C17, C21: value 10uF -> 100nF; device common:C-EU0805 -> rcl:C-EUC0402; OC_DIGIKEY 1276-2399-1-ND -> 478-7888-1-ND
- C18, C26: value 22uF -> 100nF; device common:C-EU1206 -> rcl:C-EUC0402; OC_DIGIKEY 445-6001-1-ND -> 478-7888-1-ND
- C19: value 2.2uF -> 100nF; device common:C-EU0603 -> rcl:C-EUC0402; OC_DIGIKEY 1276-1878-1-ND -> 478-7888-1-ND
- C2: value 10nF -> 10uF; device common:C-EU0402 -> rcl:C-EUC1206; OC_DIGIKEY 478-7867-1-ND -> 490-5525-1-ND
- C20: value 10uF -> 100nF; device common:C-EU1206 -> rcl:C-EUC0402; OC_DIGIKEY 490-5525-1-ND -> 478-7888-1-ND
- C23: value 10uF -> 10µF; device common:C-EU1206 -> rcl:C-EUC0805; OC_DIGIKEY 490-5525-1-ND -> 1276-2399-1-ND
- C24: value 100nF -> 10nF; OC_DIGIKEY 478-7888-1-ND -> 478-7867-1-ND
- C25: value 1uF -> 1µF; device common:C-EU0805 -> rcl:C-EUC0603; OC_DIGIKEY 490-1691-1-ND -> 490-1543-1-ND
- C27: value 1uF -> 100nF; device common:C-EU0805 -> rcl:C-EUC0402; OC_DIGIKEY 490-1691-1-ND -> 478-7888-1-ND
- C28: value 100nF -> 56pF; device common:C-EU0402 -> rcl:C-EUC0402; OC_DIGIKEY 478-7888-1-ND -> 490-1288-1-ND
- C29, C44: value 1µF -> 56pF; device common:C-EU0402 -> rcl:C-EUC0402; OC_DIGIKEY 1276-1076-1-ND -> 490-1288-1-ND
- C3: value 1µF -> 10uF; device common:C-EU0402 -> rcl:C-EUC1206; OC_DIGIKEY 1276-1076-1-ND -> 490-5525-1-ND
- C31, C32: value 1nF -> 100nF; device common:C-EU0402 -> rcl:C-EUC0402; OC_DIGIKEY 490-6348-1-ND -> 478-7888-1-ND
- C34: value 100nF -> 1µF; device common:C-EU0402 -> rcl:C-EUC0603; OC_DIGIKEY 478-7888-1-ND -> 490-1543-1-ND
- C36: value 100nF -> 10µF; device common:C-EU0402 -> rcl:C-EUC0805; OC_DIGIKEY 478-7888-1-ND -> 1276-2399-1-ND
- C37, C38: value 10nF -> 1µF; device common:C-EU0402 -> rcl:C-EUC0603; OC_DIGIKEY 478-7867-1-ND -> 490-1543-1-ND
- C4: value 100nF -> 22uF; device common:C-EU0402 -> rcl:C-EUC1206; OC_DIGIKEY 478-7888-1-ND -> 445-6001-1-ND
- C40: value 100nF -> 1nF; device common:C-EU0402 -> rcl:C-EUC0402; OC_DIGIKEY 478-7888-1-ND -> 490-6348-1-ND
- C43: value 56pF -> 10nF; device common:C-EU0402 -> rcl:C-EUC0402; OC_DIGIKEY 490-1288-1-ND -> 478-7867-1-ND
- C45: device common:C-EU0402 -> rcl:C-EUC0603; OC_DIGIKEY 1276-1076-1-ND -> 490-1543-1-ND
- C46, C47: value 56pF -> 1µF; device common:C-EU0402 -> rcl:C-EUC0603; OC_DIGIKEY 490-1288-1-ND -> 490-1543-1-ND
- C48: value 5.6pF -> 1nF; device common:C-EU0402 -> rcl:C-EUC0402; OC_DIGIKEY 490-6250-1-ND -> 490-6348-1-ND
- C49: value 4.7µF -> 100nF; device common:C-EU0603 -> rcl:C-EUC0402; OC_DIGIKEY 1276-1905-1-ND -> 478-7888-1-ND
- C5: value 56pF -> 1µF; device common:C-EU0402 -> rcl:C-EUC0805; OC_DIGIKEY 490-1288-1-ND -> 490-1691-1-ND
- C50: value 56pF -> 100nF; device common:C-EU0402 -> rcl:C-EUC0402; OC_DIGIKEY 490-1288-1-ND -> 478-7888-1-ND
- C51, C60: value 3.3pF -> 10nF; device common:C-EU0402 -> rcl:C-EUC0402; OC_DIGIKEY 490-6238-1-ND -> 478-7867-1-ND
- C52: value 10nF -> 100nF; device common:C-EU0402 -> rcl:C-EUC0402; OC_DIGIKEY 478-7867-1-ND -> 478-7888-1-ND
- C53: value 150pF -> 1µF; device common:C-EU0402 -> rcl:C-EUC0603; OC_DIGIKEY 311-1025-1-ND -> 490-1543-1-ND
- C54: value 22pF -> 1µF; device common:C-EU0402 -> rcl:C-EUC0603; OC_DIGIKEY 490-11382-1-ND -> 490-1543-1-ND
- C55: value 1nF -> 56pF; device common:C-EU0402 -> rcl:C-EUC0402; OC_DIGIKEY 490-6348-1-ND -> 490-1288-1-ND
- C56: value 33pF -> 56pF; device common:C-EU0402 -> rcl:C-EUC0402; OC_DIGIKEY 490-5936-1-ND -> 490-1288-1-ND
- C57: value 3.3pF -> 5.6pF; device common:C-EU0402 -> rcl:C-EUC0402; OC_DIGIKEY 490-6238-1-ND -> 490-6250-1-ND
- C58: value 7.5pF -> 4.7µF; device common:C-EU0402 -> rcl:C-EUC0603; OC_DIGIKEY 490-8227-1-ND -> 1276-1905-1-ND
- C59: value 1.5pF -> 3.3pF; device common:C-EU0402 -> rcl:C-EUC0402; OC_DIGIKEY 490-6212-1-ND -> 490-6238-1-ND
- C6: value 56pF -> 2.2uF; device common:C-EU0402 -> rcl:C-EUC0603; OC_DIGIKEY 490-1288-1-ND -> 1276-1878-1-ND
- C61: value 5.1pF -> 56pF; device common:C-EU0402 -> rcl:C-EUC0402; OC_DIGIKEY 490-8215-1-ND -> 490-1288-1-ND
- C62: value 2.7pF -> 150pF; device common:C-EU0402 -> rcl:C-EUC0402; OC_DIGIKEY 490-6229-1-ND -> 311-1025-1-ND
- C63: value 5.1pF -> 22pF; device common:C-EU0402 -> rcl:C-EUC0402; OC_DIGIKEY 490-8215-1-ND -> 490-11382-1-ND
- C64: value 56pF -> 1nF; device common:C-EU0402 -> rcl:C-EUC0402; OC_DIGIKEY 490-1288-1-ND -> 490-6348-1-ND
- D1, D2, D3, D4: value LED -> RCLAMP0531T; device common:LED -> LoRa Gateway:RCLAMP0531T; OC_DIGIKEY 160-1463-1-ND -> RCLAMP0531TTCTCT-ND
- D5, D6: value LED -> BAT54XV2T1G; device common:LED -> LoRa Gateway:BAT54XV2T1G; OC_DIGIKEY 160-1463-1-ND -> BAT54XV2T1GOSCT-ND
- D7: value BAT54XV2T1G -> LXES15AAA1-153; device LoRa Gateway:BAT54XV2T1G -> LoRa Gateway:LXES15AAA1-153; OC_DIGIKEY BAT54XV2T1GOSCT-ND -> 490-13210-1-ND
- FB5: device LoRa Gateway:BLM18PG121SH1D -> LoRa Gateway:BLM15PG100SN1D0402; OC_DIGIKEY 490-7815-1-ND -> 490-5976-1-ND
- L10, L11, L3, L4, L5, L6, L7, L8, L9: device common:L-EU0402 -> LoRa Gateway:L-EU0402
- R1: value 10k -> 0R; OC_DIGIKEY 541-10KJCT-ND -> 541-4062-1-ND
- R10: value 100 -> 10k; device common:R-EU0402 -> rcl:R-EU_R0402; OC_DIGIKEY 541-100ATCT-ND -> 541-10KJCT-ND
- R11, R14: value 470 -> 100; device common:R-EU0603 -> rcl:R-EU_R0402; OC_DIGIKEY 311-470GRCT-ND -> 541-100ATCT-ND
- R12, R4: value EXB-N8V101JX -> 10k; device LoRa Gateway:EXB-N8V101JX -> rcl:R-EU_R0402; OC_DIGIKEY Y10101CT-ND -> 541-10KJCT-ND
- R13: value EXB-N8V101JX -> 100; device LoRa Gateway:EXB-N8V101JX -> rcl:R-EU_R0402; OC_DIGIKEY Y10101CT-ND -> 541-100ATCT-ND
- R15: value 470 -> 0; device common:R-EU0603 -> rcl:R-EU_R0402; OC_DIGIKEY 311-470GRCT-ND -> 541-4062-1-ND
- R16: value 10k -> 470; device common:R-EU0402 -> rcl:R-EU_R0402; OC_DIGIKEY 541-10KJCT-ND -> 311-470JRCT-ND
- R17: value 10k -> 470; device common:R-EU0402 -> rcl:R-EU_R0402; OC_DIGIKEY 311-100KJRCT-ND -> 311-470JRCT-ND
- R18: value 16k -> 100; device common:R-EU0402 -> rcl:R-EU_R0402; OC_DIGIKEY 541-10KJCT-ND -> 541-100ATCT-ND
- R19: value 12k -> 100; device common:R-EU0402 -> rcl:R-EU_R0402; OC_DIGIKEY 541-10KJCT-ND -> 541-100ATCT-ND
- R2: value 100 -> 0R; device common:R-EU0402 -> rcl:R-EU_R0402; OC_DIGIKEY 541-100ATCT-ND -> 541-4062-1-ND
- R20: value 100 -> EXB-N8V101JX; device common:R-EU0402 -> LoRa Gateway:EXB-N8V101JX; OC_DIGIKEY 541-100ATCT-ND -> Y10101CT-ND
- R21: value 300 -> EXB-N8V101JX; device common:R-EU0402 -> LoRa Gateway:EXB-N8V101JX; OC_DIGIKEY RMCF0402FT300RCT-ND -> Y10101CT-ND
- R22: value 18 -> 100; device common:R-EU0402 -> rcl:R-EU_R0402; OC_DIGIKEY A129606CT-ND -> 541-100ATCT-ND
- R23: device common:R-EU0402 -> rcl:R-EU_R0402
- R24: value 49R9 -> 18; device common:R-EU0402 -> rcl:R-EU_R0402; OC_DIGIKEY 541-3967-1-ND -> A129606CT-ND
- R25: value 49R9 -> 300; device common:R-EU0402 -> rcl:R-EU_R0402; OC_DIGIKEY 541-3967-1-ND -> RMCF0402FT300RCT-ND
- R3: value 100 -> 1k; device common:R-EU0402 -> rcl:R-EU_R0402; OC_DIGIKEY 541-100ATCT-ND -> 541-1.0KJCT-ND
- R5: value 0 -> 10k; device common:R-EU0402 -> rcl:R-EU_R0402; OC_DIGIKEY 541-4062-1-ND -> 311-100KJRCT-ND
- R8: value 470 -> 100k; OC_DIGIKEY 311-470JRCT-ND -> 311-100KJRCT-ND
- R9: value 470 -> 100k; device common:R-EU0603 -> rcl:R-EU_R0402; OC_DIGIKEY 311-470GRCT-ND -> 311-100KJRCT-ND
- U1: value (none) -> SC283; device LoRa Gateway:SX1308 -> LoRa Gateway:SC283; OC_DIGIKEY SX1308IMLTRTCT-ND -> SC283WLCT-ND
- U2: value FGPMMOPA6H -> SC560H; device LoRa Gateway:FGPMMOPA6H -> LoRa Gateway:SC560H; OC_DIGIKEY (none) -> SC560HULCT-ND
- U4: value SC283 -> STM32F401CDU6; device LoRa Gateway:SC283 -> LoRa Gateway:STM32F401CDU6; OC_DIGIKEY SC283WLCT-ND -> 497-17427-ND
- U5: value SC560H -> (none); device LoRa Gateway:SC560H -> LoRa Gateway:SX1308; OC_DIGIKEY SC560HULCT-ND -> SX1308IMLTRTCT-ND
- U6, U7: OC_DIGIKEY SX1257IWLTRTCT-ND -> SX1257IWLTRTCT-ND
- X1: value END4825A -> USB2-MICRO; device LoRa Gateway:END4825A -> LoRa Gateway:USB2-MICRO; OC_DIGIKEY 644-1329-1-ND -> 609-4052-1-ND
- X2: value SMA-KE11 -> MCU Prog Header; device LoRa Gateway:SMA-KE11 -> con-amp-micromatch:MICROMATCH-6; DIGIKEY (none) -> A99463TR-ND; OC_DIGIKEY 931-1175-ND -> A30729TR-ND
- X3: value END4263A -> END4825A; device LoRa Gateway:END4263A -> LoRa Gateway:END4825A; OC_DIGIKEY 644-1328-1-ND -> 644-1329-1-ND
- X4: value SMA-KE11 -> END4263A; device LoRa Gateway:SMA-KE11 -> LoRa Gateway:END4263A; OC_DIGIKEY 931-1175-ND -> 644-1328-1-ND
Connections:
- removed net GPSRX: J1.TXD0/GPIO14, U2.RX
- removed net GPSTX: J1.RXD0/GPIO15, U2.TX
- removed net N$11: R4.7, U1.HOST_MISO
- removed net N$42: D2.A, R7.2
- removed net N$66: D4.A, R11.2
- removed net N$68: D5.A, R14.2
- removed net N$69: D6.A, R15.2
- removed net N$7: R15.1, U1.GPIO[0]
- removed net N$71: R9.1, U1.GPIO[3]
- removed net N$72: R8.2, U2.3DFIX
- removed net N$76: D1.A, R8.1
- removed net N$8: R11.1, U1.GPIO[2]
- removed net Q1_VCC: C2.1, FB1.2, X1.SBY, X1.VCC
- removed net V+: C13.1, J1.3V3@1, U2.!RESET, U2.VCC
- new net +3V3: C15.1, C16.1, C17.1, C18.1, C19.1, C20.1, C21.1, FB6.2, R9.2, S1.1, U4.VBAT, U4.VDD@1, U4.VDD@2, U4.VDD@3, U4.VDDA/VREF+
- new net 133M_OUT_EN: R10.2, U4.PB2, X3.SBY
- new net BOOT0: R8.2, S1.2, U4.BOOT0
- new net CLKO_B_32M: R22.2, U4.PH0-OSC_IN
- new net D+: D4.1, R2.1, X1.D+
- new net D-: D3.1, R1.1, X1.D-
- new net GPIO0: U4.PB1, U5.GPIO[0]
- new net GPIO2: U4.PA2, U5.GPIO[2]
- new net GPIO3: U4.PA8, U5.GPIO[3]
- new net I2C1_SCL: U4.PB7
- new net I2C1_SDA: U4.PB6
- new net N$16: C24.1, FB7.2, X3.VCC
- new net N$6: D1.1, FB3.1, X1.GND
- new net N$9: FB1.2, X1.SHIELD
- new net NRST: C13.1, R9.1, S2.2, U4.NRST, X2-1.S
- new net RADIO2_RST: U4.PA10
- new net SPI2_MISO: U4.PB14
- new net SPI2_MOSI: U4.PB15
- new net SPI2_NSS: U4.PB12
- new net SPI2_SCK: U4.PB13
- new net SWCLK: U4.PA14, X2-4.S
- new net SWDIO: U4.PA13, X2-6.S
- new net TRACESWO: U4.PB3, X2-2.S
- new net USB_DM: R1.2, U4.PA11
- new net USB_DP: R2.2, U4.PA12
- new net VBUS: D2.1, FB2.1, X1.VCC
- new net VCAP: C14.1, U4.VCAP1
- net +5V: now also C2.1, C3.1, C5.2, C6.1, FB2.2, R3.2, R4.1, R5.1, U1.CTL0A, U1.CTL0B, U1.CTL1A, U1.CTL2A, U1.CTL3A, U1.CTL3B, U1.VINA, U1.VINB, U2.VIN, U4.PA9; no longer C19.1, C20.1, C23.1, J1.5V0@1, J1.5V0@2, R16.1, R17.1, U4.CTL0A, U4.CTL0B, U4.CTL1A, U4.CTL2A, U4.CTL3A, U4.CTL3B, U4.VINA, U4.VINB, U5.VIN
- net CLKHS: now also R15.2, U5.CLKHS; no longer R5.2, U1.CLKHS
- net CLKI: now also R18.2, U6.CLK_IN; no longer R6.2, U7.CLK_IN
- net CLKO_B: now also R19.2, R22.1, U7.CLK_OUT; no longer R10.2, U6.CLK_OUT
- net FEM_EN: now also C22.1, IC1.EN, R11.1; no longer R20.2
- net GND: now also C31.2, C32.2, C33.2, C34.2, C35.2, C36.2, C37.2, C38.2, C41.1, C42.1, C43.1, C46.2, C47.2, C49.1, C5.1, C50.1, C51.1, C64.2, C65.2, C66.2, C67.2, C69.2, C70.2, C71.2, C72.2, C74.2, C75.2, D1.2, D2.2, D3.2, D4.2, D7.2, FB1.1, FB3.2, IC1.GND, JP1.6, P1.C, P2.C, P3.C, R10.1, R12.1, R21.1, R21.7, R21.8, R25.2, R26.1, R27.1, R8.1, S2.1, U1.CTL1B, U1.CTL2B, U1.GNDA@1, U1.GNDA@2, U1.GNDA@3, U1.GNDB@1, U1.GNDB@2, U1.GNDB@3, U2.GND, U4.VSS@1, U4.VSS@2, U4.VSS@3, U4.VSS@4, U4.VSSA/VREF-, U5.GND@1, U5.GND@2, U5.NC@1, U5.NC@2, U5.NC@3, U5.NC@4, U5.NC@5, U5.SCANMODE, U5.SP_VALID, U5.VSS@1, U5.VSS@2, U5.VSS@3, U5.VSS@4, U5.VSS@5, U5.VSS@6, U5.VSS@7, U5.VSS@8, U5.VSS@9, U7.I_IN, U7.Q_IN, X2-3.S, X4.GND@1, X5.GND; no longer C33.1, C34.1, C35.1, C36.1, C37.1, C38.1, C40.2, C41.2, C42.2, C43.2, C48.2, C49.2, C5.2, C55.2, C56.2, C61.2, D1.C, D2.C, D3.C, D4.C, D5.C, D6.C, D9.2, J1.GND@1, J1.GND@2, J1.GND@3, J1.GND@4, J1.GND@5, J1.GND@6, J1.GND@7, J1.GND@8, R1.1, R13.1, R13.2, R13.7, R13.8, R19.1, R24.1, R25.1, U1.GND@1, U1.GND@2, U1.NC@1, U1.NC@2, U1.NC@3, U1.NC@4, U1.NC@5, U1.SCANMODE, U1.SP_VALID, U1.VSS@1, U1.VSS@2, U1.VSS@3, U1.VSS@4, U1.VSS@5, U1.VSS@6, U1.VSS@7, U1.VSS@8, U1.VSS@9, U10.N/C@6, U2.GND@1, U2.GND@2, U2.GND@3, U2.GND@4, U3.GND, U4.CTL1B, U4.CTL2B, U4.GNDA@1, U4.GNDA@2, U4.GNDA@3, U4.GNDB@1, U4.GNDB@2, U4.GNDB@3, U5.GND, U6.I_IN, U6.Q_IN, X1.GND, X2.GND, X3.GND@1
- net IRXD_A: now also R20.5, U6.I_OUT; no longer R12.5, U7.I_OUT
- net IRXD_B: now also R21.5, U7.I_OUT; no longer R13.5, U6.I_OUT
- net ITXD_A: now also R20.7, U6.I_IN; no longer R12.7, U7.I_IN
- net LNA_EN: now also C28.1, R13.1; no longer C5.1, R2.1
- net MISO_A: now also U5.RADIO_A_MISO, U6.MISO; no longer U1.RADIO_A_MISO, U7.MISO
- net MISO_B: now also U5.RADIO_B_MISO, U7.MISO; no longer U1.RADIO_B_MISO, U6.MISO
- net MOSI_A: now also U5.RADIO_A_MOSI, U6.MOSI; no longer U1.RADIO_A_MOSI, U7.MOSI
- net MOSI_B: now also U5.RADIO_B_MOSI, U7.MOSI; no longer U1.RADIO_B_MOSI, U6.MOSI
- net N$1: now also U1.LXA; no longer U4.LXA
- net N$10: now also P1.A, R3.1; no longer R4.8, U1.HOST_SCK
- net N$12: now also C7.1, FB4.2, IC1.VIN; no longer C17.1, FB3.2, U3.EN, U3.VIN
- net N$13: now also C74.1, U6.VR_ANA2; no longer C40.1, U7.VR_ANA2
- net N$14: now also P2.A, R16.2; no longer R4.6, U1.HOST_MOSI
- net N$15: now also P3.A, R17.2; no longer R13.3, U1.B_QI_RX
- net N$17: now also R15.1, X3.OUT; no longer R5.1, X1.OUT
- net N$18: now also C39.1, FB9.2, X4.VCC; no longer C28.1, FB4.2, X3.VCC
- net N$19: now also R27.2; no longer R25.2
- net N$2: now also U1.LXB; no longer U4.LXB
- net N$22: now also R26.2; no longer R24.2
- net N$23: now also C63.1; no longer C54.1
- net N$24: now also C67.1, C70.1; no longer C58.1, C61.1
- net N$25: now also C62.1; no longer C53.1
- net N$27: now also C68.2, C69.1; no longer C59.2, C60.1
- net N$28: now also R13.2, U5.LNA_A_CTRL; no longer R2.2, U1.LNA_A_CTRL
- net N$29: now also R14.2, U5.PA_A_CTRL; no longer R3.2, U1.PA_A_CTRL
- net N$3: now also C75.1, IC1.NR; no longer R18.1, R19.2, U3.FB
- net N$31: now also C72.1; no longer C63.1
- net N$32: now also C65.1, C68.1; no longer C57.1, C59.1
- net N$33: now also R11.2, U4.PB0; no longer R4.5, U1.HOST_CSN
- net N$34: now also C71.1, C73.1, D7.1; no longer C62.1, C64.1, D9.1
- net N$35: now also C59.1; no longer C51.1
- net N$36: now also C61.2; no longer C50.2
- net N$37: now also C59.2, R24.1, R25.1; no longer C51.2, R22.1, R23.1
- net N$38: now also C31.1, U5.VCC18@3; no longer C9.1, U1.VCC18@3
- net N$39: now also R23.1, R24.2; no longer R21.1, R22.2
- net N$4: now also C8.1, U2.BYP; no longer C24.1, U5.BYP
- net N$40: now also C55.2; no longer C46.2
- net N$41: now also C61.1; no longer C50.1
- net N$43: now also C56.2, C57.1; no longer C47.2, C48.1
- net N$44: now also C56.1; no longer C47.1
- net N$45: now also R18.1, U5.SP_CLK_OUT; no longer D3.A, R9.2
- net N$46: now also C55.1, U6.RF_OP; no longer C46.1, U7.RF_OP
- net N$47: now also C52.1, U7.VR_ANA2; no longer C39.1, U6.VR_ANA2
- net N$48: now also D6.C, U7.RESET; no longer D7.C, U6.RESET
- net N$49: now also C48.1, U7.XTB; no longer C31.1, U6.XTB
- net N$5: now also C12.1, FB5.1, X2-5.S; no longer R6.1, U1.SP_CLK_OUT
- net N$50: now also R21.3, U5.B_QI_RX; no longer R13.4, U1.B_IQ_RX
- net N$51: now also R21.4, U5.B_IQ_RX; no longer U2.EX_ANT, X2.1
- net N$52: now also C40.1, U6.XTB; no longer C32.1, U7.XTB
- net N$53: now also C43.2, U6.VR_PA; no longer C38.2, U7.VR_PA
- net N$54: now also C51.2, U7.VR_PA; no longer C37.2, U6.VR_PA
- net N$55: now also C50.2, U7.VR_ANA1; no longer C35.2, U6.VR_ANA1
- net N$56: now also C49.2, U7.VR_DIG; no longer C33.2, U6.VR_DIG
- net N$57: now also C42.2, U6.VR_ANA1; no longer C36.2, U7.VR_ANA1
- net N$58: now also R19.1, U5.CLK32M; no longer R10.1, U1.CLK32M
- net N$59: now also R20.4, U5.A_IQ_RX; no longer R12.4, U1.A_IQ_RX
- net N$60: now also R20.3, U5.A_QI_RX; no longer R12.3, U1.A_QI_RX
- net N$61: now also R20.2, U5.A_IQ_TX; no longer R12.2, U1.A_IQ_TX
- net N$62: now also R20.1, U5.A_QI_TX; no longer R12.1, U1.A_QI_TX
- net N$63: now also C41.2, U6.VR_DIG; no longer C34.2, U7.VR_DIG
- net N$64: now also C44.1, U6.RF_ON; no longer C43.1, U7.RF_ON
- net N$65: now also C73.2, X5.1; no longer C64.2, X4.1
- net N$67: now also C33.1, C34.1, U5.VCC33@2; no longer C11.1, C12.1, U1.VCC33@2
- net N$70: now also D5.C, U6.RESET; no longer D8.C, U7.RESET
- net NSS_A: now also U5.RADIO_A_CS, U6.NSS; no longer U1.RADIO_A_CS, U7.NSS
- net NSS_B: now also U5.RADIO_B_CS, U7.NSS; no longer U1.RADIO_B_CS, U6.NSS
- net PA_EN: now also C29.1, R14.1; no longer C6.1, R3.1
- net PPS: now also U4.PB10, U5.GPS_IN; no longer J1.GEN5/GPIO24, U1.GPS_IN, U2.PPS
- net QRXD_A: now also R20.6, U6.Q_OUT; no longer R12.6, U7.Q_OUT
- net QRXD_B: now also R21.6, U7.Q_OUT; no longer R13.6, U6.Q_OUT
- net QTXD_A: now also R20.8, U6.Q_IN; no longer R12.8, U7.Q_IN
- net RADIO_EN_A: now also R4.2, U2.ENA, U4.PB8; no longer R16.2, U5.ENA
- net RADIO_EN_B: now also R5.2, U2.ENB, U4.PB9; no longer R17.2, U5.ENB
- net RADIO_RST: now also D5.A, D6.A, U4.PA0; no longer D7.A, D8.A, U1.RADIO_RST
- net RESET: now also JP1.1, R12.2, U4.PA3, U5.RESET; no longer J1.GEN/6GPIO25, R1.2, U1.RESET
- net RX_ON: now also R17.1, U4.PB5, U5.GPIO[1]; no longer R14.1, U1.GPIO[1]
- net SCK_A: now also U5.RADIO_A_SCK, U6.SCK; no longer U1.RADIO_A_SCK, U7.SCK
- net SCK_B: now also U5.RADIO_B_SCK, U7.SCK; no longer U1.RADIO_B_SCK, U6.SCK
- net SPI_MISO: now also JP1.4, U4.PA6, U5.HOST_MISO; no longer J1.GPIO9/MISO, R4.2
- net SPI_MOSI: now also JP1.5, U4.PA7, U5.HOST_MOSI; no longer J1.GPIO10/MOSI, R4.3
- net SPI_NSS: now also JP1.2, U4.PA4, U5.HOST_CSN; no longer J1.!CE0!/GPIO8, R4.4
- net SPI_SCK: now also JP1.3, U4.PA5, U5.HOST_SCK; no longer J1.GPIO11/SCLK, R4.1
- net TX_ON: now also R16.1, U4.PB4, U5.GPIO[4]; no longer R7.1, U1.GPIO[4]
- net VCC: now also C36.1, C4.1, FB8.1, U1.VOUTB; no longer C14.1, C26.1, FB2.1, U4.VOUTB
- net VCCA_A: now also C38.1, C46.1, C60.1, C9.1, FB9.1, U2.OUTA, U6.VBAT1, U6.VBAT2, U6.VBAT3; no longer C25.1, C30.1, C42.1, C52.1, FB4.1, U5.OUTA, U7.VBAT1, U7.VBAT2, U7.VBAT3
- net VCCA_B: now also C11.1, C47.1, C53.1, C54.1, U2.OUTB, U7.VBAT1, U7.VBAT2, U7.VBAT3; no longer C27.1, C29.1, C41.1, C44.1, U5.OUTB, U6.VBAT1, U6.VBAT2, U6.VBAT3
- net VCCDIG18: now also C25.1, C26.1, C27.1, C30.1, C35.1, C37.1, FB8.2, U5.VCC18@1, U5.VCC18@2, U5.VCC18@4, U5.VCC18@5; no longer C15.1, C16.1, C3.1, C4.1, C7.1, C8.1, FB2.2, U1.VCC18@1, U1.VCC18@2, U1.VCC18@4, U1.VCC18@5
- net VCCDIG33: now also C23.1, C32.1, FB4.1, FB5.2, FB6.1, FB7.1, U1.VOUTA, U5.VCC33@1; no longer C10.1, C18.1, FB1.1, FB3.1, U1.VCC33@1, U4.VOUTA
- net VCCINT: now also C10.1, FB10.1, IC1.SNS, IC1.VOUT; no longer C21.1, C22.1, FB5.1, R18.2, R20.1, U3.VOUT
- net VCC_FEM: now also C58.1, C64.1, C66.1, FB10.2; no longer C49.1, C55.1, C56.1, FB5.2
- net XTL_OUT: now also C40.2, C48.2, X4.OUT; no longer C31.2, C32.2, X3.OUT
